File: Eagle/Net Widget.brd (EAGLE design)
At the start: 66 x 45.7 mm, 13 parts, among them IC1 ATmega1284P

Commit message: Match pin numbers to WildFire; route.
Parts:
- moved C4 1.59 mm to (33.0, 34.9)
Connections:
- net CARD_CS: now also IC1.24; no longer IC1.21
- net CS: now also IC1.40; no longer IC1.22
- net TFT_CS: now also IC1.12; no longer IC1.40
- net TFT_RESET: now also IC1.13; no longer IC1.41
- net VBEN: now also IC1.41; no longer IC1.23
Routing:
- net CS: track 76.6 -> 19.7 mm, vias 0 -> 2
- net VBEN: track 81.7 -> 36.7 mm
- net TFT_CS: track 21.9 -> 59.9 mm, vias 1 -> 3
- net RESET: track 64.0 -> 97.5 mm, vias 2 -> 0
- net GND: track 121.0 -> 153.7 mm, vias 1 -> 5
- net MISO: track 78.4 -> 49.8 mm, vias 2 -> 3
- net RX: track 38.5 -> 17.2 mm
- net CARD_CS: track 71.5 -> 56.6 mm
- net TFT_RESET: track 38.3 -> 52.8 mm
- net D/C: track 39.3 -> 25.0 mm
- net MOSI: track 60.1 -> 49.6 mm, vias 2 -> 3
- net VCC: track 150.5 -> 142.7 mm, vias 5 -> 3
- net SCK: track 51.0 -> 57.0 mm, vias 3 -> 2
- net LITE: track 28.0 -> 25.6 mm, vias 1 -> 3
- net IRQ: track 21.0 -> 22.0 mm, vias 2 -> 0
Other:
- board text added: "March 7, 2015"
- board text removed: "February 20, 2015"
